File: KiCAD/OUTPUT_ADAPTER_BOARD/ADAPTER_BOARD.kicad_pcb (KiCad board)
At the start: 2 copper layers, 58 x 107 mm, 81 parts, among them Q1 Q_NPN_CBE, Q10 Q_NPN_CBE, Q11 Q_NPN_CBE, Q12 Q_NPN_CBE, Q13 Q_NPN_CBE, Q14 Q_NPN_CBE, Q15 Q_NPN_CBE, Q16 Q_NPN_CBE, Q17 Q_NPN_CBE, Q18 Q_NPN_CBE, Q19 Q_NPN_CBE, Q2 Q_NPN_CBE, Q20 Q_NPN_CBE, Q21 Q_NPN_CBE, Q22 Q_NPN_CBE, Q23 Q_NPN_CBE, Q24 Q_NPN_CBE, Q3 Q_NPN_CBE, Q4 Q_NPN_CBE, Q5 Q_NPN_CBE, Q6 Q_NPN_CBE, Q7 Q_NPN_CBE, Q8 Q_NPN_CBE, Q9 Q_NPN_CBE

Commit message: Text label updates.
Other:
- board text added: "Vidas Simkus vic.simkus@simkus.com https://www.simkus.com"
Changed lines of the file:
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@@
   )
   (gr_text "Vidas Simkus (vic.simkus@simkus.com)\nhttps://www.simkus.com" (at 55.8 75.2 270) (layer B.SilkS)
-    (effects (font (size 1.3 1.3) (thickness 0.2)) (justify mirror))
+    (effects (font (size 2 2) (thickness 0.3)) (justify mirror))
   )
-  (gr_text "Vidas Simkus (vic.simkus@simkus.com)\nhttps://www.simkus.com" (at 79.1 124.4) (layer F.SilkS)
-    (effects (font (size 1.3 1.3) (thickness 0.2)))
+  (gr_text "Vidas Simkus\nvic.simkus@simkus.com\nhttps://www.simkus.com" (at 79.61 124.64) (layer F.SilkS)
+    (effects (font (size 1.9 1.9) (thickness 0.35)))
   )
   (gr_text 12 (at 106 75.059991) (layer F.SilkS)

Commit message: V2 of the board.
Parts:
- moved VDC24 3.52 mm to (102.7, 39.8)
- moved PLC24 0.25 mm to (105.6, 81.7)
Routing:
- net GND: track 5.91 -> 3.04 mm, vias 567 -> 636
- net /P17: track 36.6 -> 37.2 mm
Other:
- board text added: "PN: GOUT"
- board text added: "Vidas Simkus -- https://www.simkus.com"
- board text removed: "Vidas Simkus (vic.simkus@simkus.com) https://www.simkus.com"
- board text removed: "Vidas Simkus vic.simkus@simkus.com https://www.simkus.com"
