File: KiCAD/INPUT_ADAPTER_BOARD/OUTPUT_CONNECTORS.sch (KiCad schematic (older format))
At the start: 14 parts

Commit message: Footprint updates.
Connections:
- net P01: now also JP12.1 (A)
- net P02: no longer JP12.1 (A)
- net P03: now also JP11.1 (A)
- net P04: no longer JP11.1 (A)
- net P05: now also JP10.1 (A)
- net P06: no longer JP10.1 (A)
- net P07: now also JP9.1 (A)
- net P08: no longer JP9.1 (A)
- net P09: now also JP8.1 (A)
- net P10: no longer JP8.1 (A)
- net P11: now also JP7.1 (A)
- net P12: no longer JP7.1 (A)
- net P13: now also JP6.1 (A)
- net P14: no longer JP6.1 (A)
- net P15: now also JP5.1 (A)
- net P16: no longer JP5.1 (A)
- net P17: now also JP4.1 (A)
- net P18: no longer JP4.1 (A)
- net P19: now also JP3.1 (A)
- net P20: no longer JP3.1 (A)
- net P21: now also JP2.1 (A)
- net P22: no longer JP2.1 (A)
- net P23: now also JP1.1 (A)
- net P24: no longer JP1.1 (A)
Other:
- moved on the sheet: JP1, JP10, JP11, JP12, JP2, JP3, JP4, JP5, JP6, JP7, JP8, JP9
